Commit message: hier: dual arm configuration

File: crisp_controllers_robot_demos/config/fr3/fr3.ros2_control.urdf.xacro (robot description, xacro)
@@ -19,5 +19,5 @@
           <param name="version">1.0.0</param>
           <param name="robot_type">${robot_type}</param>
-          <param name="prefix">${arm_prefix}</param>
+          <param name="prefix">${arm_prefix_modified}</param>
           <xacro:unless value="${use_fake_hardware}">
             <plugin>franka_hardware/FrankaHardwareInterface</plugin>
@@ -44,11 +44,11 @@
         </joint>
       </xacro:macro>
-      <xacro:configure_joint joint_name="${arm_prefix}${robot_type}_joint1" initial_position="0.0"/>
-      <xacro:configure_joint joint_name="${arm_prefix}${robot_type}_joint2" initial_position="${-pi/4}"/>
-      <xacro:configure_joint joint_name="${arm_prefix}${robot_type}_joint3" initial_position="0.0"/>
-      <xacro:configure_joint joint_name="${arm_prefix}${robot_type}_joint4" initial_position="${-3*pi/4}"/>
-      <xacro:configure_joint joint_name="${arm_prefix}${robot_type}_joint5" initial_position="0.0"/>
-      <xacro:configure_joint joint_name="${arm_prefix}${robot_type}_joint6" initial_position="${pi/2}"/>
-      <xacro:configure_joint joint_name="${arm_prefix}${robot_type}_joint7" initial_position="${pi/4}"/>
+      <xacro:configure_joint joint_name="${arm_prefix_modified}${robot_type}_joint1" initial_position="0.0"/>
+      <xacro:configure_joint joint_name="${arm_prefix_modified}${robot_type}_joint2" initial_position="${-pi/4}"/>
+      <xacro:configure_joint joint_name="${arm_prefix_modified}${robot_type}_joint3" initial_position="0.0"/>
+      <xacro:configure_joint joint_name="${arm_prefix_modified}${robot_type}_joint4" initial_position="${-3*pi/4}"/>
+      <xacro:configure_joint joint_name="${arm_prefix_modified}${robot_type}_joint5" initial_position="0.0"/>
+      <xacro:configure_joint joint_name="${arm_prefix_modified}${robot_type}_joint6" initial_position="${pi/2}"/>
+      <xacro:configure_joint joint_name="${arm_prefix_modified}${robot_type}_joint7" initial_position="${pi/4}"/>
     </ros2_control>
   </xacro:macro>

File: crisp_controllers_robot_demos/config/fr3/fr3.urdf.xacro (robot description, xacro)
@@ -29,5 +29,5 @@
                       gazebo_effort="${gazebo_effort}"
                       no_prefix="${no_prefix}"
-                      arm_prefix="${arm_prefix}"
+                      arm_prefix="${arm_prefix_modified}"
                       connected_to="${arm_prefix_modified}base">
   </xacro:franka_robot>

File: crisp_controllers_robot_demos/config/fr3/fr3_dual.urdf.xacro (robot description, xacro)
@@ -30,9 +30,9 @@
   <joint name="left_base_to_world_joint" type="fixed"> <parent link="world"/>
     <child link="left_base"/>
-    <origin rpy="0 0 0" xyz="0 0 0"/>
+    <origin rpy="-0.7854 0 0" xyz="0 0.1065 0"/>
   </joint>
   <joint name="right_base_to_world_joint" type="fixed"> <parent link="world"/>
     <child link="right_base"/>
-    <origin rpy="0 0 0" xyz="0 1.0 0"/>
+    <origin rpy="0.7854 0 0" xyz="0 -0.1065 0"/>
   </joint>
 </robot>

File: crisp_controllers_robot_demos/config/fr3/fr3_single.urdf.xacro (robot description, xacro)
@@ -25,4 +25,6 @@
   <!-- Type of Franka arm -->
   <xacro:arg name="robot_type" default="fr3" />
+  <!-- Fixed mounting preset for multi-arm setups -->
+  <xacro:arg name="mounting" default="none" />
   <xacro:arg name="has_camera" default="false" />
 <xacro:property name="arm_prefix_modified" value="${'' if xacro.arg('arm_prefix') == '' else xacro.arg('arm_prefix') + '_'}" />
@@ -35,3 +37,19 @@
     hand="$(arg load_gripper)"
   />
+  <xacro:if value="${xacro.arg('mounting') == 'dual_left'}">
+    <link name="world"/>
+    <joint name="left_base_to_world_joint" type="fixed">
+      <parent link="world"/>
+      <child link="left_base"/>
+      <origin rpy="-0.7854 0 0" xyz="0 0.1065 0"/>
+    </joint>
+  </xacro:if>
+  <xacro:if value="${xacro.arg('mounting') == 'dual_right'}">
+    <link name="world"/>
+    <joint name="right_base_to_world_joint" type="fixed">
+      <parent link="world"/>
+      <child link="right_base"/>
+      <origin rpy="0.7854 0 0" xyz="0 -0.1065 0"/>
+    </joint>
+  </xacro:if>
 </robot>
